File: 3V3_5V/3V3_5V.kicad_sch (KiCad schematic)
At the start: 32 parts, among them J101 USB_C_Receptacle_PowerOnly_6P, J102 Conn_01x02_Pin, J103 Conn_01x02_Pin, U101 LTM4644EY-1-PBF

Commit message: edit schematic and PCB layout
Parts:
- removed C101, C102, C103, C104, C110, C111: C, symbol Device:C
- removed R106, R108: 60.4k, Resistor_SMD:R_0603_1608Metric, symbol Device:R
- removed R107, R109: 13.3k, Resistor_SMD:R_0603_1608Metric, symbol Device:R
- C102: renamed from C105; value 220uF -> 47uF
- C103: renamed from C106; value 220uF -> 47uF
- C104: renamed from C107; value 10uF -> 22uF
- C105: renamed from C108; value 10uF -> 22uF
- C107: renamed from C113; value 220uF -> 47uF
- C108: renamed from C114; value 220uF -> 47uF
- C109: renamed from C115; value 10uF -> 22uF
- C110: renamed from C116; value 10uF -> 22uF
- C111: renamed from C109; value C -> 1n; footprint (none) -> Capacitor_SMD:C_0603_1608Metric
- C112: value C -> 1n; footprint (none) -> Capacitor_SMD:C_0603_1608Metric
- renumbered C117 to C101, C118 to C106, R104 to R103, R103 to R104
Connections:
- net COMP2 is gone; now on net COMP: U101.H7 (COMP3), U101.L7 (COMP4)
- net GND: now also C111.2, C112.2
- net TR1/SS1: now also C111.1, C112.1
- net INTVcc1: now reaches U101.C4 (INTVCC1)
- net INTVcc1: now also U101.F4 (INTVCC2)
- net COMP1 renamed COMP
- net PG3 renamed PG2
- no-connect marks 0 -> 2
Other:
- moved on the sheet: C111

Commit message: add to sch and pcb
Connections:
- net 3V3B is gone; now on net +3.3VB: R103.1
Changed lines of the file:
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@@
+		)
+	)
+	(label "3V3B"
+		(at 251.46 66.04 0)
+		(fields_autoplaced yes)
+		(effects
+			(font
+				(size 1.27 1.27)
+			)
+			(justify left bottom)
 		)
 	)
